File: Raspberry/Raspberry.kicad_pcb (KiCad board)
At the start: 2 copper layers, 9 parts, among them J1 Conn_01x02_Pin, J2 Conn_01x04, J3 Conn_01x02_Pin

Commit message: Actualización de la PCB, carpeta de campo
Parts:
- removed C1: 100nF, Capacitor_SMD:C_0805_2012Metric
- removed J1: Conn_01x02_Pin, Connector_JST:JST_PH_B2B-PH-K_1x02_P2.00mm_Vertical
- removed the R1 at (161.5, 94.5)
- removed the R2 at (161.5, 98.5)
- added R3: 22K, Resistor_THT:R_Axial_DIN0204_L3.6mm_D1.6mm_P7.62mm_Horizontal, F.Cu at (146.8, 106.0)
- added R4: 10K, Resistor_THT:R_Axial_DIN0204_L3.6mm_D1.6mm_P7.62mm_Horizontal, F.Cu at (139.2, 101.0)
- added R5: 220, Resistor_THT:R_Axial_DIN0204_L3.6mm_D1.6mm_P7.62mm_Horizontal, F.Cu at (139.4, 95.0)
- A1: footprint Module:RaspberryPi_Pico_W_SMD_HandSolder -> Module:RaspberryPi_Pico_Common_THT
- R1: renamed from R3; value 30K -> 22K; footprint Resistor_THT:R_Axial_DIN0207_L6.3mm_D2.5mm_P2.54mm_Vertical -> Resistor_THT:R_Axial_DIN0204_L3.6mm_D1.6mm_P7.62mm_Horizontal
- R2: renamed from R4; footprint Resistor_THT:R_Axial_DIN0207_L6.3mm_D2.5mm_P2.54mm_Vertical -> Resistor_THT:R_Axial_DIN0204_L3.6mm_D1.6mm_P7.62mm_Horizontal
- moved J3 56.1 mm to (140.0, 61.0), turned to -90 degrees
- moved A1 27.1 mm to (114.3, 80.5)
- moved R2 24.8 mm to (139.2, 117.5)
- moved R1 17.1 mm to (146.5, 111.0), turned to 180 degrees
- moved J2 15.1 mm to (142.0, 80.4), turned to -90 degrees
Connections:
- A1 pad 33: Earth -> unconnected-(A1-AGND-Pad33)
- A1 pad 40: unconnected-(A1-VBUS-Pad40) -> VBUS y R5
- J2 pad 3: +3.3V -> VBUS
- J3 pad 1: J3 -> R1 y R3
- R1 pad 1: J3 -> J3 (1)
Routing:
- net GP7: track 0.82 -> 75.6 mm
- net GP6: track 0.00 -> 64.7 mm
- net ADC0: track 0.00 -> 19.4 mm
- net VBUS: track 0.00 -> 16.0 mm
- net ADC1: track 0.00 -> 12.3 mm
- net J3 (1): track 0.00 -> 5.11 mm
- added copper zone on B.Cu, net Earth
Other:
- board outline added: 50 x 100 mm
- board text added: "7° 1° AVC"
- board text added: "PL.E.PE.R 2025"
